File: schematic.kicad_sch (KiCad schematic)
At the start: 43 parts, among them J1 SLB4-G-21, J2 SLB4-G-22, J3 MKDS5/2-9.5, J4 MKDS5/2-9.5, J5 DVM_Connector, Q1 2N3904, Q2 STF7NM80

Commit message: Fix schematic vs SVG discrepancies: net name, diode refs, value strings
- Rename global net GATE → GATE_CTRL to match reference SVG
- Correct D2/D3/D4 reference designators to match SVG bridge labelling
  (D1 was already correct; D2↔D3 and D3↔D4 swapped)
- Add voltage to zener value fields: D9 BZX85C12 12V, D_LED BZX55C8V2 8.2V,
  D_Vcc 1N4744A 15V
- Add Vf to LED1 value: RED 5mm Vf~2V
- Add ratings to Q2 value: STF7NM80 800V 6A
- Add power rating to all 100kΩ/0.6W resistors (R3, R_LED1–3, R_sig1–5,
  R_sig_bot): 100k → 100k 0.6W

Co-Authored-By: Claude Sonnet 4.6 <noreply@anthropic.com>
Parts:
- D9: value BZX85C12 -> BZX85C12 12V
- D_LED: value BZX55C8V2 -> BZX55C8V2 8.2V
- D_Vcc: value 1N4744A -> 1N4744A 15V
- LED1: value RED 5mm -> RED 5mm Vf~2V
- Q2: value STF7NM80 -> STF7NM80 800V 6A
- R3, R_LED1, R_LED2, R_LED3, R_sig1, R_sig2, R_sig3, R_sig4, R_sig5, R_sig_bot: value 100k -> 100k 0.6W
- renumbered D4 to D2, D2 to D3, D3 to D4
Connections:
- net GATE renamed GATE_CTRL
