File: KiCAD/hv_section.kicad_sch (KiCad schematic)
At the start: 15 parts, among them J1 SLB4-G-21, J2 SLB4-G-22, J3 MKDS5/2-9.5, J4 MKDS5/2-9.5, Q2 STF7NM80

Commit message: Update Q2 to STP10NK80Z across schematics, SVG, and CSV
- KiCAD/hv_section.kicad_sch: Q2 value STF7NM80 → STP10NK80Z
- KiCAD/CapacitorDischarger.kicad_sch: Q2 value updated to STP10NK80Z 800V 9A
- blocks/gen_full_schematic.py: branch 2 comment updated
- blocks/full_schematic.svg: regenerated with STP10NK80Z label
- TO_BUY_list.csv: Q2 primary updated to STP10NK80Z

Simulation files retain STF7NM80 SPICE model — functionally equivalent.

Co-Authored-By: Claude Sonnet 4.6 <noreply@anthropic.com>
Parts:
- Q2: value STF7NM80 -> STP10NK80Z
Changed lines of the file:
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@@
     (instances (project "CapacitorDischarger" (path "/a1000000-0001-0001-0001-000000000001" (reference "R_fast") (unit 1))))
   )
-  ;; Q2 — MOSFET STF7NM80, D at top (drain connected to R_fast bottom), S at bottom → GND
+  ;; Q2 — MOSFET STP10NK80Z, D at top (drain connected to R_fast bottom), S at bottom → GND
   (symbol
     (lib_id "Device:Q_NMOS_GDS")
     (at 160 80 0) (unit 1) (in_bom yes) (on_board yes)
     (property "Reference" "Q2" (at 165 78 0) (effects (font (size 1.27 1.27))))
-    (property "Value" "STF7NM80" (at 165 80.5 0) (effects (font (size 1.27 1.27))))
+    (property "Value" "STP10NK80Z" (at 165 80.5 0) (effects (font (size 1.27 1.27))))
     (property "Footprint" "Package_TO_SOT_THT:TO-220-3_Vertical" (at 0 0 0) (effects (font (size 1.27 1.27)) hide))
     (property "Datasheet" "" (at 0 0 0) (effects (font (size 1.27 1.27)) hide))

Commit message: Fix footprints to match KiCad 10 library and actual sourced components
Five footprint names didn't exist in KiCad 10 (caused 'Cannot add' errors),
and R_slow/R_fast were sized for generic ceramics, not the actual Ohmite parts.

Library name fixes (all three schematics):
  R_Axial_Power_L15mm_W5mm_P20.32mm   → R_Axial_DIN0516_L15.5mm_D5.0mm_P20.32mm_Horizontal
  C_Disc_D3.8mm_W2.6mm_P5.00mm        → C_Disc_D3.8mm_W2.6mm_P2.50mm
  CP_Radial_D4.0mm_P2.50mm            → CP_Radial_D4.0mm_P2.00mm
  Potentiometer_Vishay_T93_Vertical    → Potentiometer_Bourns_3296W_Vertical

Correct sizing for sourced Ohmite wirewound resistors:
  R_slow1-5 (Ohmite 45F, 5W, body 23.8×8.7mm) → R_Axial_Power_L25.0mm_W9.0mm_P30.48mm
  R_fast     (Ohmite 27J, 7W, body 32.1×10mm)  → R_Axial_Power_L38.0mm_W9.0mm_P40.64mm

Co-Authored-By: Claude Sonnet 4.6 <noreply@anthropic.com>
Parts:
- R_fast: footprint Resistor_THT:R_Axial_Power_L38mm_W10mm_P41.91mm -> Resistor_THT:R_Axial_Power_L38.0mm_W9.0mm_P40.64mm
- R_slow1, R_slow2, R_slow3, R_slow4, R_slow5: footprint Resistor_THT:R_Axial_Power_L38mm_W10mm_P41.91mm -> Resistor_THT:R_Axial_Power_L25.0mm_W9.0mm_P30.48mm
Changed lines of the file:
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@@
     (property "Reference" "R_slow1" (at 123 45 0) (effects (font (size 1.27 1.27)) (justify left)))
     (property "Value" "4k7 5W" (at 123 47.5 0) (effects (font (size 1.27 1.27)) (justify left)))
-    (property "Footprint" "Resistor_THT:R_Axial_Power_L38mm_W10mm_P41.91mm" (at 0 0 0) (effects (font (size 1.27 1.27)) hide))
+    (property "Footprint" "Resistor_THT:R_Axial_Power_L25.0mm_W9.0mm_P30.48mm" (at 0 0 0) (effects (font (size 1.27 1.27)) hide))
     (property "Datasheet" "" (at 0 0 0) (effects (font (size 1.27 1.27)) hide))
     (pin "1")
@@
     (property "Reference" "R_slow2" (at 123 62 0) (effects (font (size 1.27 1.27)) (justify left)))
     (property "Value" "4k7 5W" (at 123 64.5 0) (effects (font (size 1.27 1.27)) (justify left)))
-    (property "Footprint" "Resistor_THT:R_Axial_Power_L38mm_W10mm_P41.91mm" (at 0 0 0) (effects (font (size 1.27 1.27)) hide))
+    (property "Footprint" "Resistor_THT:R_Axial_Power_L25.0mm_W9.0mm_P30.48mm" (at 0 0 0) (effects (font (size 1.27 1.27)) hide))
     (property "Datasheet" "" (at 0 0 0) (effects (font (size 1.27 1.27)) hide))
     (pin "1")
@@
     (property "Reference" "R_slow3" (at 123 79 0) (effects (font (size 1.27 1.27)) (justify left)))
     (property "Value" "4k7 5W" (at 123 81.5 0) (effects (font (size 1.27 1.27)) (justify left)))
-    (property "Footprint" "Resistor_THT:R_Axial_Power_L38mm_W10mm_P41.91mm" (at 0 0 0) (effects (font (size 1.27 1.27)) hide))
+    (property "Footprint" "Resistor_THT:R_Axial_Power_L25.0mm_W9.0mm_P30.48mm" (at 0 0 0) (effects (font (size 1.27 1.27)) hide))
     (property "Datasheet" "" (at 0 0 0) (effects (font (size 1.27 1.27)) hide))
     (pin "1")
@@
     (property "Reference" "R_slow4" (at 123 96 0) (effects (font (size 1.27 1.27)) (justify left)))
     (property "Value" "4k7 5W" (at 123 98.5 0) (effects (font (size 1.27 1.27)) (justify left)))
-    (property "Footprint" "Resistor_THT:R_Axial_Power_L38mm_W10mm_P41.91mm" (at 0 0 0) (effects (font (size 1.27 1.27)) hide))
+    (property "Footprint" "Resistor_THT:R_Axial_Power_L25.0mm_W9.0mm_P30.48mm" (at 0 0 0) (effects (font (size 1.27 1.27)) hide))
     (property "Datasheet" "" (at 0 0 0) (effects (font (size 1.27 1.27)) hide))
     (pin "1")
@@
     (property "Reference" "R_slow5" (at 123 113 0) (effects (font (size 1.27 1.27)) (justify left)))
     (property "Value" "4k7 5W" (at 123 115.5 0) (effects (font (size 1.27 1.27)) (justify left)))
-    (property "Footprint" "Resistor_THT:R_Axial_Power_L38mm_W10mm_P41.91mm" (at 0 0 0) (effects (font (size 1.27 1.27)) hide))
+    (property "Footprint" "Resistor_THT:R_Axial_Power_L25.0mm_W9.0mm_P30.48mm" (at 0 0 0) (effects (font (size 1.27 1.27)) hide))
     (property "Datasheet" "" (at 0 0 0) (effects (font (size 1.27 1.27)) hide))
     (pin "1")
@@
     (property "Reference" "R_fast" (at 163 55 0) (effects (font (size 1.27 1.27)) (justify left)))
     (property "Value" "50R 5W" (at 163 57.5 0) (effects (font (size 1.27 1.27)) (justify left)))
-    (property "Footprint" "Resistor_THT:R_Axial_Power_L38mm_W10mm_P41.91mm" (at 0 0 0) (effects (font (size 1.27 1.27)) hide))
+    (property "Footprint" "Resistor_THT:R_Axial_Power_L38.0mm_W9.0mm_P40.64mm" (at 0 0 0) (effects (font (size 1.27 1.27)) hide))
     (property "Datasheet" "" (at 0 0 0) (effects (font (size 1.27 1.27)) hide))
     (pin "1")

Commit message: Fix symbol lib_ids and inner sub-symbol names for KiCad 10 compatibility
Schematic was generated with lib_ids that don't exist in KiCad 10,
causing 'symbol not found' on Update from Library and 'invalid symbol'
errors on sub-symbol name mismatches.

lib_id renames (pin numbers were already correct):
  Device:R_Large    → Device:R
  Device:R_POT      → Device:R_Potentiometer_Trim
  Device:CP         → Device:C_Polarized
  Device:Q_NPN_BCE  → Transistor_BJT:MPSA42  (E=1, B=2, C=3)
  Device:Q_NMOS_GDS → Transistor_FET:Q_NMOS_GDS  (G=1, D=2, S=3)

Inner sub-symbol names updated to match new lib_ids:
  CP_0/1_1 → C_Polarized_0/1_1
  R_POT_0/1_1 → R_Potentiometer_Trim_0/1_1
  Q_NPN_BCE_0/1_1 → MPSA42_0/1_1
  R_Large_0/1_1 → R_0/1_1 (duplicate Device:R entry removed)

Applied to all three schematic files.

Co-Authored-By: Claude Sonnet 4.6 <noreply@anthropic.com>
Parts:
- Q2: symbol Device:Q_NMOS_GDS -> Transistor_FET:Q_NMOS_GDS
- R_fast, R_slow1, R_slow2, R_slow3, R_slow4, R_slow5: symbol Device:R_Large -> Device:R
Changed lines of the file:
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@@
   ;; ═══════════════════════════════════════════════════════════════════════
   (symbol
-    (lib_id "Device:R_Large")
+    (lib_id "Device:R")
     (at 120 45 0) (unit 1) (in_bom yes) (on_board yes)
     (property "Reference" "R_slow1" (at 123 45 0) (effects (font (size 1.27 1.27)) (justify left)))
@@
   )
   (symbol
-    (lib_id "Device:R_Large")
+    (lib_id "Device:R")
     (at 120 62 0) (unit 1) (in_bom yes) (on_board yes)
     (property "Reference" "R_slow2" (at 123 62 0) (effects (font (size 1.27 1.27)) (justify left)))
@@
   )
   (symbol
-    (lib_id "Device:R_Large")
+    (lib_id "Device:R")
     (at 120 79 0) (unit 1) (in_bom yes) (on_board yes)
     (property "Reference" "R_slow3" (at 123 79 0) (effects (font (size 1.27 1.27)) (justify left)))
@@
   )
   (symbol
-    (lib_id "Device:R_Large")
+    (lib_id "Device:R")
     (at 120 96 0) (unit 1) (in_bom yes) (on_board yes)
     (property "Reference" "R_slow4" (at 123 96 0) (effects (font (size 1.27 1.27)) (justify left)))
@@
   )
   (symbol
-    (lib_id "Device:R_Large")
+    (lib_id "Device:R")
     (at 120 113 0) (unit 1) (in_bom yes) (on_board yes)
     (property "Reference" "R_slow5" (at 123 113 0) (effects (font (size 1.27 1.27)) (justify left)))
@@
   ;; ═══════════════════════════════════════════════════════════════════════
   (symbol
-    (lib_id "Device:R_Large")
+    (lib_id "Device:R")
     (at 160 55 0) (unit 1) (in_bom yes) (on_board yes)
     (property "Reference" "R_fast" (at 163 55 0) (effects (font (size 1.27 1.27)) (justify left)))
@@
   ;; Q2 — MOSFET STP10NK80Z, D at top (drain connected to R_fast bottom), S at bottom → GND
   (symbol
-    (lib_id "Device:Q_NMOS_GDS")
+    (lib_id "Transistor_FET:Q_NMOS_GDS")
     (at 160 80 0) (unit 1) (in_bom yes) (on_board yes)
     (property "Reference" "Q2" (at 165 78 0) (effects (font (size 1.27 1.27))))

Commit message: Design review fixes: fuse F1, battery-powered DVM, R3=10k, KiCad polarity fixes
Review of the full design (schematic, BOM, simulations) surfaced and fixed:

- Add F1 protection fuse (2A/600V KLKD002.T + Keystone 3517 clips) in
  series after the bridge — opens on single-fault Q2-stuck-on (~12A).
- Reduce R3 100k -> 10k: Q1 threshold now hFE-independent, 63V nominal /
  68V at the BF=40 corner (was 76V / 154V, peak I_fast ~3A over the 2A
  PCB limit).
- Replace the DVM Vcc parasitic dropper (4x15k + 1N4744A) with a 9V
  battery (BT1, holder w/ switch) via new polarized JST XH input J6:
  the sourced DVM module measures 12-15mA, beyond the dropper's 9.75mA.
- Fix gate-drive drawing in the generated schematic: D9 is a shunt clamp
  at GATE_CTRL, not in series (SVG previously showed a broken topology).
- KiCad root schematic: bridge D1-D4 and LED1 were mounted reversed —
  rotated 180 (netlist-verified); F1 and J6 added, dropper removed,
  VCC_DVM rail unshorted from node_sig, C_byp1 pins actually connected;
  value fields R3/R5/R_fast corrected; section drafts updated to match.
- Simulations: bridge D1-D4 now modeled (residual ~1V verified), MOSFET
  model renamed to STP10NK80Z, low-hFE threshold corner scenario G2
  added, Vcc branch removed with the dropper; suite passes 8/8.
- BOM/README: regenerate stale bom.md (Q1=MPSA42, 4x R_LED, 10k R_cal),
  correct stress-math notes, document residual voltage, threshold range,
  discharge time 45.5s @ 600V/1mF, and high-efficiency LED requirement.

Co-Authored-By: Claude Fable 5 <noreply@anthropic.com>
Parts:
- added F1: 2A/600V, Fuse:Fuseholder_Cylinder-10x38mm, symbol Device:Fuse
- R_fast: value 50R 5W -> 50R 7W
Connections:
- net HV+: now also F1.2; no longer D1.K, D2.K, D3.K
- new net: D1.K, D2.K, D3.K, F1.1
Changed lines of the file:
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@@
     (at 160 55 0) (unit 1) (in_bom yes) (on_board yes)
     (property "Reference" "R_fast" (at 163 55 0) (effects (font (size 1.27 1.27)) (justify left)))
-    (property "Value" "50R 5W" (at 163 57.5 0) (effects (font (size 1.27 1.27)) (justify left)))
+    (property "Value" "50R 7W" (at 163 57.5 0) (effects (font (size 1.27 1.27)) (justify left)))
     (property "Footprint" "Resistor_THT:R_Axial_Power_L38.0mm_W9.0mm_P40.64mm" (at 0 0 0) (effects (font (size 1.27 1.27)) hide))
     (property "Datasheet" "" (at 0 0 0) (effects (font (size 1.27 1.27)) hide))
@@
     (instances (project "CapacitorDischarger" (path "/a1000000-0001-0001-0001-000000000001" (reference "#PWR04") (unit 1))))
   )
+  ;; F1 — protection fuse, 2A/600V (KLKD002.T, 10.3×38mm + Keystone 3517 clips)
+  ;; In series in the HV+ line between bridge cathodes and the HV+ bus:
+  ;; opens on single-fault (Q1 open / D9 fail → Q2 full-on at 600V → ~12A).
+  ;; Horizontal at (87, 45): pin1 at (83.19, 45), pin2 at (90.81, 45)
+  (symbol
+    (lib_id "Device:Fuse")
+    (at 87 45 0) (unit 1) (in_bom yes) (on_board yes)
+    (property "Reference" "F1" (at 87 40 0) (effects (font (size 1.27 1.27))))
+    (property "Value" "2A/600V" (at 87 42.5 0) (effects (font (size 1.27 1.27))))
+    (property "Footprint" "Fuse:Fuseholder_Cylinder-10x38mm" (at 0 0 0) (effects (font (size 1.27 1.27)) hide))
+    (property "Datasheet" "" (at 0 0 0) (effects (font (size 1.27 1.27)) hide))
+    (pin "1")
+    (pin "2")
+    (instances (project "CapacitorDischarger" (path "/a1000000-0001-0001-0001-000000000001" (reference "F1") (unit 1))))
+  )
   ;; GND at J4 pin2 (20, 93.27)
   (symbol
@@
   ;; D1 K = (63.81, 45), D3 K = (78.81, 45) — both cathodes meet at HV+ bus
   (wire (pts (xy 63.81 45) (xy 78.81 45)) (stroke (width 0) (type default)) (uuid "w0024"))
-  ;; HV+ bus right to R_slow1 pin1 (120, 41.19)
-  (wire (pts (xy 78.81 45) (xy 100 45)) (stroke (width 0) (type default)) (uuid "w0025"))
+  ;; Bridge cathodes → F1 pin1; F1 pin2 → HV+ bus (fuse in series)
+  (wire (pts (xy 78.81 45) (xy 83.19 45)) (stroke (width 0) (type default)) (uuid "w0025"))
+  (wire (pts (xy 90.81 45) (xy 100 45)) (stroke (width 0) (type default)) (uuid "w0025b"))
   (wire (pts (xy 100 45) (xy 120 41.19)) (stroke (width 0) (type default)) (uuid "w0026"))
   ;; HV+ bus branch to R_fast pin1
