File: KiCAD/lv_section.kicad_sch (KiCad schematic)
At the start: 28 parts, among them J5 DVM_Connector, Q1 2N3904

Commit message: Replace Q1 2N3904→MPSA42, add R_LED4, swap R_cal to 10kΩ 3296W
- Q1: 2N3904 (40V) → MPSA42 (300V) — safe margin in 600V circuit
- R_LED: 3→4 resistors in series; each now sees ≤150V (was ~200V, 80% of rating)
- R_cal: 200kΩ wirewound → 10kΩ cermet 25-turn (3296W-1-103LF); previous
  value could overdrive DVM beyond its 100V input limit
- Add 3386P-1-103LF as sourced_unused
- All 7 simulation scenarios PASS with updated MPSA42 model and R_LED4 node

Co-Authored-By: Claude Sonnet 4.6 <noreply@anthropic.com>
Parts:
- added R_LED4: 100k, Resistor_THT:R_Axial_DIN0207_L6.3mm_D2.5mm_P10.16mm_Horizontal, symbol Device:R
- Q1: value 2N3904 -> MPSA42
- R_cal: value 200k trim -> 10k trim
Connections:
- net at R_LED3.2: now also R_LED4.1; no longer D_LED.A
- new net: D_LED.A, R_LED4.2
Changed lines of the file:
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@@
     (instances (project "CapacitorDischarger" (path "/b2000000-0002-0002-0002-000000000002" (reference "R3") (unit 1))))
   )
-  ;; Q1 — 2N3904 NPN, at (90, 52)
+  ;; Q1 — MPSA42 NPN, at (90, 52)
   ;; B at (87.46, 52); C at (90.508, 46.92); E at (90.508, 57.08)
   (symbol
@@
     (at 90 52 0) (unit 1) (in_bom yes) (on_board yes)
     (property "Reference" "Q1" (at 95 50 0) (effects (font (size 1.27 1.27))))
-    (property "Value" "2N3904" (at 95 52.5 0) (effects (font (size 1.27 1.27))))
+    (property "Value" "MPSA42" (at 95 52.5 0) (effects (font (size 1.27 1.27))))
     (property "Footprint" "Package_TO_SOT_THT:TO-92_Inline" (at 0 0 0) (effects (font (size 1.27 1.27)) hide))
     (property "Datasheet" "" (at 0 0 0) (effects (font (size 1.27 1.27)) hide))
@@
   ;; ═══════════════════════════════════════════════════════════════════════
   ;; BLOCK C — LED DANGER INDICATOR
-  ;; HV+ → R_LED1 → R_LED2 → R_LED3 → D_LED(K) D_LED(A) → LED1(A) LED1(K) → GND
+  ;; HV+ → R_LED1 → R_LED2 → R_LED3 → R_LED4 → D_LED(K) D_LED(A) → LED1(A) LED1(K) → GND
   ;; Column x=152, top at y=25
   ;; ═══════════════════════════════════════════════════════════════════════
@@
     (instances (project "CapacitorDischarger" (path "/b2000000-0002-0002-0002-000000000002" (reference "R_LED3") (unit 1))))
   )
-  ;; D_LED — BZX55C8V2 (8.2V Zener), K-up at (152, 73)
-  ;; angle=270 → K at (152, 69.19); A at (152, 76.81)
+  ;; R_LED4 at (152, 71)
+  ;; pin1 at (152, 68.46); pin2 at (152, 73.54)
+  (symbol
+    (lib_id "Device:R")
+    (at 152 71 0) (unit 1) (in_bom yes) (on_board yes)
+    (property "Reference" "R_LED4" (at 155 71 0) (effects (font (size 1.27 1.27)) (justify left)))
+    (property "Value" "100k" (at 155 73.5 0) (effects (font (size 1.27 1.27)) (justify left)))
+    (property "Footprint" "Resistor_THT:R_Axial_DIN0207_L6.3mm_D2.5mm_P10.16mm_Horizontal" (at 0 0 0) (effects (font (size 1.27 1.27)) hide))
+    (property "Datasheet" "" (at 0 0 0) (effects (font (size 1.27 1.27)) hide))
+    (pin "1")
+    (pin "2")
+    (instances (project "CapacitorDischarger" (path "/b2000000-0002-0002-0002-000000000002" (reference "R_LED4") (unit 1))))
+  )
+  ;; D_LED — BZX55C8V2 (8.2V Zener), K-up at (152, 85)
+  ;; angle=270 → K at (152, 81.19); A at (152, 88.81)
   (symbol
     (lib_id "Device:D_Zener")
-    (at 152 73 270) (unit 1) (in_bom yes) (on_board yes)
-    (property "Reference" "D_LED" (at 155 71 0) (effects (font (size 1.27 1.27))))
-    (property "Value" "BZX55C8V2" (at 155 73.5 0) (effects (font (size 1.27 1.27))))
+    (at 152 85 270) (unit 1) (in_bom yes) (on_board yes)
+    (property "Reference" "D_LED" (at 155 83 0) (effects (font (size 1.27 1.27))))
+    (property "Value" "BZX55C8V2" (at 155 85.5 0) (effects (font (size 1.27 1.27))))
     (property "Footprint" "Diode_THT:D_DO-35_SOD27_P7.62mm_Horizontal" (at 0 0 0) (effects (font (size 1.27 1.27)) hide))
     (property "Datasheet" "" (at 0 0 0) (effects (font (size 1.27 1.27)) hide))
@@
     (instances (project "CapacitorDischarger" (path "/b2000000-0002-0002-0002-000000000002" (reference "D_LED") (unit 1))))
   )
-  ;; LED1 — red 5mm, D_LED (K-up at 152,88), angle=270 → K at (152,84.19); A at (152,91.81)
+  ;; LED1 — red 5mm, angle=270 → K at (152,96.19); A at (152,103.81)
   (symbol
     (lib_id "Device:LED")
-    (at 152 88 270) (unit 1) (in_bom yes) (on_board yes)
-    (property "Reference" "LED1" (at 155 86 0) (effects (font (size 1.27 1.27))))
-    (property "Value" "RED 5mm" (at 155 88.5 0) (effects (font (size 1.27 1.27))))
+    (at 152 100 270) (unit 1) (in_bom yes) (on_board yes)
+    (property "Reference" "LED1" (at 155 98 0) (effects (font (size 1.27 1.27))))
+    (property "Value" "RED 5mm" (at 155 100.5 0) (effects (font (size 1.27 1.27))))
     (property "Footprint" "LED_THT:LED_D5.0mm" (at 0 0 0) (effects (font (size 1.27 1.27)) hide))
     (property "Datasheet" "" (at 0 0 0) (effects (font (size 1.27 1.27)) hide))
@@
     (instances (project "CapacitorDischarger" (path "/b2000000-0002-0002-0002-000000000002" (reference "LED1") (unit 1))))
   )
-  ;; GND at LED1 anode bottom (152, 96)
+  ;; GND at LED1 anode bottom (152, 110)
   (symbol
     (lib_id "power:GND")
-    (at 152 98 0) (unit 1) (in_bom yes) (on_board yes)
-    (property "Reference" "#PWR04" (at 152 104 0) (effects (font (size 1.27 1.27)) hide))
-    (property "Value" "GND" (at 152 101 0) (effects (font (size 1.27 1.27))))
+    (at 152 110 0) (unit 1) (in_bom yes) (on_board yes)
+    (property "Reference" "#PWR04" (at 152 116 0) (effects (font (size 1.27 1.27)) hide))
+    (property "Value" "GND" (at 152 113 0) (effects (font (size 1.27 1.27))))
     (pin "1")
     (instances (project "CapacitorDischarger" (path "/b2000000-0002-0002-0002-000000000002" (reference "#PWR04") (unit 1))))
@@
     (instances (project "CapacitorDischarger" (path "/b2000000-0002-0002-0002-000000000002" (reference "R_sig_bot") (unit 1))))
   )
-  ;; R_cal — 200kΩ trimmer, R_POT at (185, 113)
+  ;; R_cal — 10kΩ trimmer (3296W), R_POT at (185, 113)
   ;; pin1 at (185, 109.19); pin2 at (185, 116.81) → GND; wiper shorted to pin1 (no-connect acceptable)
   (symbol
@@
     (at 185 113 0) (unit 1) (in_bom yes) (on_board yes)
     (property "Reference" "R_cal" (at 190 113 0) (effects (font (size 1.27 1.27)) (justify left)))
-    (property "Value" "200k trim" (at 190 115.5 0) (effects (font (size 1.27 1.27)) (justify left)))
+    (property "Value" "10k trim" (at 190 115.5 0) (effects (font (size 1.27 1.27)) (justify left)))
     (property "Footprint" "Potentiometer_THT:Potentiometer_Vishay_T93_Vertical" (at 0 0 0) (effects (font (size 1.27 1.27)) hide))
     (property "Datasheet" "" (at 0 0 0) (effects (font (size 1.27 1.27)) hide))
@@
   (wire (pts (xy 152 37.54) (xy 152 44.46)) (stroke (width 0) (type default)) (uuid "lw0021"))
   (wire (pts (xy 152 49.54) (xy 152 56.46)) (stroke (width 0) (type default)) (uuid "lw0022"))
-  ;; R_LED3 pin2 → D_LED K (at 152,69.19)
-  (wire (pts (xy 152 61.54) (xy 152 69.19)) (stroke (width 0) (type default)) (uuid "lw0023"))
-  ;; D_LED A → LED1 K (D_LED A at 152,76.81; LED1 K at 152,84.19)
-  (wire (pts (xy 152 76.81) (xy 152 84.19)) (stroke (width 0) (type default)) (uuid "lw0024"))
-  ;; LED1 A → GND (LED1 A at 152,91.81)
-  (wire (pts (xy 152 91.81) (xy 152 98)) (stroke (width 0) (type default)) (uuid "lw0025"))
+  ;; R_LED3 pin2 → R_LED4 pin1
+  (wire (pts (xy 152 61.54) (xy 152 68.46)) (stroke (width 0) (type default)) (uuid "lw0023"))
+  ;; R_LED4 pin2 → D_LED K (at 152,81.19)
+  (wire (pts (xy 152 73.54) (xy 152 81.19)) (stroke (width 0) (type default)) (uuid "lw0023b"))
+  ;; D_LED A → LED1 K (D_LED A at 152,88.81; LED1 K at 152,96.19)
+  (wire (pts (xy 152 88.81) (xy 152 96.19)) (stroke (width 0) (type default)) (uuid "lw0024"))
+  ;; LED1 A → GND (LED1 A at 152,103.81)
+  (wire (pts (xy 152 103.81) (xy 152 110)) (stroke (width 0) (type default)) (uuid "lw0025"))
   ;; ═══════════════════════════════════════════════════════════════════════
   ;; WIRES — Block D (DVM divider)

Commit message: Fix footprints to match KiCad 10 library and actual sourced components
Five footprint names didn't exist in KiCad 10 (caused 'Cannot add' errors),
and R_slow/R_fast were sized for generic ceramics, not the actual Ohmite parts.

Library name fixes (all three schematics):
  R_Axial_Power_L15mm_W5mm_P20.32mm   → R_Axial_DIN0516_L15.5mm_D5.0mm_P20.32mm_Horizontal
  C_Disc_D3.8mm_W2.6mm_P5.00mm        → C_Disc_D3.8mm_W2.6mm_P2.50mm
  CP_Radial_D4.0mm_P2.50mm            → CP_Radial_D4.0mm_P2.00mm
  Potentiometer_Vishay_T93_Vertical    → Potentiometer_Bourns_3296W_Vertical

Correct sizing for sourced Ohmite wirewound resistors:
  R_slow1-5 (Ohmite 45F, 5W, body 23.8×8.7mm) → R_Axial_Power_L25.0mm_W9.0mm_P30.48mm
  R_fast     (Ohmite 27J, 7W, body 32.1×10mm)  → R_Axial_Power_L38.0mm_W9.0mm_P40.64mm

Co-Authored-By: Claude Sonnet 4.6 <noreply@anthropic.com>
Parts:
- C_Vcc: footprint Capacitor_THT:CP_Radial_D4.0mm_P2.50mm -> Capacitor_THT:CP_Radial_D4.0mm_P2.00mm
- C_byp1, C_byp2: footprint Capacitor_THT:C_Disc_D3.8mm_W2.6mm_P5.00mm -> Capacitor_THT:C_Disc_D3.8mm_W2.6mm_P2.50mm
- R1, R5, R_drop1, R_drop2, R_drop3, R_drop4: footprint Resistor_THT:R_Axial_Power_L15mm_W5mm_P20.32mm -> Resistor_THT:R_Axial_DIN0516_L15.5mm_D5.0mm_P20.32mm_Horizontal
- R_cal: footprint Potentiometer_THT:Potentiometer_Vishay_T93_Vertical -> Potentiometer_THT:Potentiometer_Bourns_3296W_Vertical
Changed lines of the file:
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@@
     (property "Reference" "R1" (at 53 40 0) (effects (font (size 1.27 1.27)) (justify left)))
     (property "Value" "1M 1W" (at 53 42.5 0) (effects (font (size 1.27 1.27)) (justify left)))
-    (property "Footprint" "Resistor_THT:R_Axial_Power_L15mm_W5mm_P20.32mm" (at 0 0 0) (effects (font (size 1.27 1.27)) hide))
+    (property "Footprint" "Resistor_THT:R_Axial_DIN0516_L15.5mm_D5.0mm_P20.32mm_Horizontal" (at 0 0 0) (effects (font (size 1.27 1.27)) hide))
     (property "Datasheet" "" (at 0 0 0) (effects (font (size 1.27 1.27)) hide))
     (pin "1")
@@
     (property "Reference" "R5" (at 111 28 0) (effects (font (size 1.27 1.27)) (justify left)))
     (property "Value" "470k 1W" (at 111 30.5 0) (effects (font (size 1.27 1.27)) (justify left)))
-    (property "Footprint" "Resistor_THT:R_Axial_Power_L15mm_W5mm_P20.32mm" (at 0 0 0) (effects (font (size 1.27 1.27)) hide))
+    (property "Footprint" "Resistor_THT:R_Axial_DIN0516_L15.5mm_D5.0mm_P20.32mm_Horizontal" (at 0 0 0) (effects (font (size 1.27 1.27)) hide))
     (property "Datasheet" "" (at 0 0 0) (effects (font (size 1.27 1.27)) hide))
     (pin "1")
@@
     (property "Reference" "R_cal" (at 190 113 0) (effects (font (size 1.27 1.27)) (justify left)))
     (property "Value" "10k trim" (at 190 115.5 0) (effects (font (size 1.27 1.27)) (justify left)))
-    (property "Footprint" "Potentiometer_THT:Potentiometer_Vishay_T93_Vertical" (at 0 0 0) (effects (font (size 1.27 1.27)) hide))
+    (property "Footprint" "Potentiometer_THT:Potentiometer_Bourns_3296W_Vertical" (at 0 0 0) (effects (font (size 1.27 1.27)) hide))
     (property "Datasheet" "" (at 0 0 0) (effects (font (size 1.27 1.27)) hide))
     (pin "1")
@@
     (property "Reference" "R_drop1" (at 233 35 0) (effects (font (size 1.27 1.27)) (justify left)))
     (property "Value" "15k 3W" (at 233 37.5 0) (effects (font (size 1.27 1.27)) (justify left)))
-    (property "Footprint" "Resistor_THT:R_Axial_Power_L15mm_W5mm_P20.32mm" (at 0 0 0) (effects (font (size 1.27 1.27)) hide))
+    (property "Footprint" "Resistor_THT:R_Axial_DIN0516_L15.5mm_D5.0mm_P20.32mm_Horizontal" (at 0 0 0) (effects (font (size 1.27 1.27)) hide))
     (property "Datasheet" "" (at 0 0 0) (effects (font (size 1.27 1.27)) hide))
     (pin "1")
@@
     (property "Reference" "R_drop2" (at 233 52 0) (effects (font (size 1.27 1.27)) (justify left)))
     (property "Value" "15k 3W" (at 233 54.5 0) (effects (font (size 1.27 1.27)) (justify left)))
-    (property "Footprint" "Resistor_THT:R_Axial_Power_L15mm_W5mm_P20.32mm" (at 0 0 0) (effects (font (size 1.27 1.27)) hide))
+    (property "Footprint" "Resistor_THT:R_Axial_DIN0516_L15.5mm_D5.0mm_P20.32mm_Horizontal" (at 0 0 0) (effects (font (size 1.27 1.27)) hide))
     (property "Datasheet" "" (at 0 0 0) (effects (font (size 1.27 1.27)) hide))
     (pin "1")
@@
     (property "Reference" "R_drop3" (at 233 69 0) (effects (font (size 1.27 1.27)) (justify left)))
     (property "Value" "15k 3W" (at 233 71.5 0) (effects (font (size 1.27 1.27)) (justify left)))
-    (property "Footprint" "Resistor_THT:R_Axial_Power_L15mm_W5mm_P20.32mm" (at 0 0 0) (effects (font (size 1.27 1.27)) hide))
+    (property "Footprint" "Resistor_THT:R_Axial_DIN0516_L15.5mm_D5.0mm_P20.32mm_Horizontal" (at 0 0 0) (effects (font (size 1.27 1.27)) hide))
     (property "Datasheet" "" (at 0 0 0) (effects (font (size 1.27 1.27)) hide))
     (pin "1")
@@
     (property "Reference" "R_drop4" (at 233 86 0) (effects (font (size 1.27 1.27)) (justify left)))
     (property "Value" "15k 3W" (at 233 88.5 0) (effects (font (size 1.27 1.27)) (justify left)))
-    (property "Footprint" "Resistor_THT:R_Axial_Power_L15mm_W5mm_P20.32mm" (at 0 0 0) (effects (font (size 1.27 1.27)) hide))
+    (property "Footprint" "Resistor_THT:R_Axial_DIN0516_L15.5mm_D5.0mm_P20.32mm_Horizontal" (at 0 0 0) (effects (font (size 1.27 1.27)) hide))
     (property "Datasheet" "" (at 0 0 0) (effects (font (size 1.27 1.27)) hide))
     (pin "1")
@@
     (property "Reference" "C_Vcc" (at 263 100 0) (effects (font (size 1.27 1.27))))
     (property "Value" "10uF 25V" (at 263 102.5 0) (effects (font (size 1.27 1.27))))
-    (property "Footprint" "Capacitor_THT:CP_Radial_D4.0mm_P2.50mm" (at 0 0 0) (effects (font (size 1.27 1.27)) hide))
+    (property "Footprint" "Capacitor_THT:CP_Radial_D4.0mm_P2.00mm" (at 0 0 0) (effects (font (size 1.27 1.27)) hide))
     (property "Datasheet" "" (at 0 0 0) (effects (font (size 1.27 1.27)) hide))
     (pin "1")
@@
     (property "Reference" "C_byp1" (at 274 100 0) (effects (font (size 1.27 1.27))))
     (property "Value" "100nF" (at 274 102.5 0) (effects (font (size 1.27 1.27))))
-    (property "Footprint" "Capacitor_THT:C_Disc_D3.8mm_W2.6mm_P5.00mm" (at 0 0 0) (effects (font (size 1.27 1.27)) hide))
+    (property "Footprint" "Capacitor_THT:C_Disc_D3.8mm_W2.6mm_P2.50mm" (at 0 0 0) (effects (font (size 1.27 1.27)) hide))
     (property "Datasheet" "" (at 0 0 0) (effects (font (size 1.27 1.27)) hide))
     (pin "1")
@@
     (property "Reference" "C_byp2" (at 122 50 0) (effects (font (size 1.27 1.27))))
     (property "Value" "100nF" (at 122 52.5 0) (effects (font (size 1.27 1.27))))
-    (property "Footprint" "Capacitor_THT:C_Disc_D3.8mm_W2.6mm_P5.00mm" (at 0 0 0) (effects (font (size 1.27 1.27)) hide))
-    (property "Datasheet" "" (at 0 0 0) (effects (font (size 1.27 1.27)) hide))
-    (pin "1")
+    (property "Footprint" "Capacitor_THT:C_Disc_D3.8mm_W2.6mm_P2.50mm" (at 0 0 0) (effects (font (size 1.27 1.27)) hide))
+    (property "Datasheet" "" (at 0 0 0) (effects (font (size 1.27 1.27)) hide))
+    (pin "1")

Commit message: Fix symbol lib_ids and inner sub-symbol names for KiCad 10 compatibility
Schematic was generated with lib_ids that don't exist in KiCad 10,
causing 'symbol not found' on Update from Library and 'invalid symbol'
errors on sub-symbol name mismatches.

lib_id renames (pin numbers were already correct):
  Device:R_Large    → Device:R
  Device:R_POT      → Device:R_Potentiometer_Trim
  Device:CP         → Device:C_Polarized
  Device:Q_NPN_BCE  → Transistor_BJT:MPSA42  (E=1, B=2, C=3)
  Device:Q_NMOS_GDS → Transistor_FET:Q_NMOS_GDS  (G=1, D=2, S=3)

Inner sub-symbol names updated to match new lib_ids:
  CP_0/1_1 → C_Polarized_0/1_1
  R_POT_0/1_1 → R_Potentiometer_Trim_0/1_1
  Q_NPN_BCE_0/1_1 → MPSA42_0/1_1
  R_Large_0/1_1 → R_0/1_1 (duplicate Device:R entry removed)

Applied to all three schematic files.

Co-Authored-By: Claude Sonnet 4.6 <noreply@anthropic.com>
Parts:
- C_Vcc: symbol Device:CP -> Device:C_Polarized
- Q1: symbol Device:Q_NPN_BCE -> Transistor_BJT:MPSA42
- R1, R5, R_drop1, R_drop2, R_drop3, R_drop4: symbol Device:R_Large -> Device:R
- R_cal: symbol Device:R_POT -> Device:R_Potentiometer_Trim
Connections:
- net GATE: no longer R5.2
- net GND: now also Q1.1 (E); no longer Q1.E
- net HV+: no longer R1.1, R5.1, R_drop1.1
- net node_A: no longer R1.2
- net node_Vcc: no longer R_drop4.2
- net at R4.2: now also Q1.3 (C); no longer Q1.C
- net at R_drop1.2: no longer R_drop2.1
- net at R_drop2.2: no longer R_drop3.1
- net at R_drop3.2: no longer R_drop4.1
Changed lines of the file:
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@@
   ;; pin1 at (50, 36.19) → HV+ bus; pin2 at (50, 43.81) → node_A
   (symbol
-    (lib_id "Device:R_Large")
+    (lib_id "Device:R")
     (at 50 40 0) (unit 1) (in_bom yes) (on_board yes)
     (property "Reference" "R1" (at 53 40 0) (effects (font (size 1.27 1.27)) (justify left)))
@@
   ;; B at (87.46, 52); C at (90.508, 46.92); E at (90.508, 57.08)
   (symbol
-    (lib_id "Device:Q_NPN_BCE")
+    (lib_id "Transistor_BJT:MPSA42")
     (at 90 52 0) (unit 1) (in_bom yes) (on_board yes)
     (property "Reference" "Q1" (at 95 50 0) (effects (font (size 1.27 1.27))))
@@
   ;; pin1 at (108, 24.19) → HV+ bus; pin2 at (108, 31.81) → GATE node
   (symbol
-    (lib_id "Device:R_Large")
+    (lib_id "Device:R")
     (at 108 28 0) (unit 1) (in_bom yes) (on_board yes)
     (property "Reference" "R5" (at 111 28 0) (effects (font (size 1.27 1.27)) (justify left)))
@@
   ;; pin1 at (185, 109.19); pin2 at (185, 116.81) → GND; wiper shorted to pin1 (no-connect acceptable)
   (symbol
-    (lib_id "Device:R_POT")
+    (lib_id "Device:R_Potentiometer_Trim")
     (at 185 113 0) (unit 1) (in_bom yes) (on_board yes)
     (property "Reference" "R_cal" (at 190 113 0) (effects (font (size 1.27 1.27)) (justify left)))
@@
   ;; ═══════════════════════════════════════════════════════════════════════
   (symbol
-    (lib_id "Device:R_Large")
+    (lib_id "Device:R")
     (at 230 35 0) (unit 1) (in_bom yes) (on_board yes)
     (property "Reference" "R_drop1" (at 233 35 0) (effects (font (size 1.27 1.27)) (justify left)))
@@
   )
   (symbol
-    (lib_id "Device:R_Large")
+    (lib_id "Device:R")
     (at 230 52 0) (unit 1) (in_bom yes) (on_board yes)
     (property "Reference" "R_drop2" (at 233 52 0) (effects (font (size 1.27 1.27)) (justify left)))
@@
   )
   (symbol
-    (lib_id "Device:R_Large")
+    (lib_id "Device:R")
     (at 230 69 0) (unit 1) (in_bom yes) (on_board yes)
     (property "Reference" "R_drop3" (at 233 69 0) (effects (font (size 1.27 1.27)) (justify left)))
@@
   )
   (symbol
-    (lib_id "Device:R_Large")
+    (lib_id "Device:R")
     (at 230 86 0) (unit 1) (in_bom yes) (on_board yes)
     (property "Reference" "R_drop4" (at 233 86 0) (effects (font (size 1.27 1.27)) (justify left)))
@@
   ;; Device:CP → pin1(+) at (260, 98.19); pin2(-) at (260, 105.81) → GND
   (symbol
-    (lib_id "Device:CP")
+    (lib_id "Device:C_Polarized")
     (at 260 102 0) (unit 1) (in_bom yes) (on_board yes)
     (property "Reference" "C_Vcc" (at 263 100 0) (effects (font (size 1.27 1.27))))

Commit message: Design review fixes: fuse F1, battery-powered DVM, R3=10k, KiCad polarity fixes
Review of the full design (schematic, BOM, simulations) surfaced and fixed:

- Add F1 protection fuse (2A/600V KLKD002.T + Keystone 3517 clips) in
  series after the bridge — opens on single-fault Q2-stuck-on (~12A).
- Reduce R3 100k -> 10k: Q1 threshold now hFE-independent, 63V nominal /
  68V at the BF=40 corner (was 76V / 154V, peak I_fast ~3A over the 2A
  PCB limit).
- Replace the DVM Vcc parasitic dropper (4x15k + 1N4744A) with a 9V
  battery (BT1, holder w/ switch) via new polarized JST XH input J6:
  the sourced DVM module measures 12-15mA, beyond the dropper's 9.75mA.
- Fix gate-drive drawing in the generated schematic: D9 is a shunt clamp
  at GATE_CTRL, not in series (SVG previously showed a broken topology).
- KiCad root schematic: bridge D1-D4 and LED1 were mounted reversed —
  rotated 180 (netlist-verified); F1 and J6 added, dropper removed,
  VCC_DVM rail unshorted from node_sig, C_byp1 pins actually connected;
  value fields R3/R5/R_fast corrected; section drafts updated to match.
- Simulations: bridge D1-D4 now modeled (residual ~1V verified), MOSFET
  model renamed to STP10NK80Z, low-hFE threshold corner scenario G2
  added, Vcc branch removed with the dropper; suite passes 8/8.
- BOM/README: regenerate stale bom.md (Q1=MPSA42, 4x R_LED, 10k R_cal),
  correct stress-math notes, document residual voltage, threshold range,
  discharge time 45.5s @ 600V/1mF, and high-efficiency LED requirement.

Co-Authored-By: Claude Fable 5 <noreply@anthropic.com>
Parts:
- removed D_Vcc: 1N4744A, Diode_THT:D_DO-41_SOD81_P10.16mm_Horizontal, symbol Device:D_Zener
- removed R_drop1, R_drop2, R_drop3, R_drop4: 15k 3W, Resistor_THT:R_Axial_DIN0516_L15.5mm_D5.0mm_P20.32mm_Horizontal, symbol Device:R
- added J6: BATT 9V, Connector_JST:JST_XH_B2B-XH-A_1x02_P2.50mm_Vertical, symbol Connector:Conn_01x02_Pin
- R3: value 100k -> 10k
- R5: value 470k 1W -> 470k 3W
Connections:
- net GND: now also J6.1 (Pin_1)
- net node_Vcc renamed VCC_DVM
- net VCC_DVM: now also J6.2 (Pin_2)
