File: KiCAD/CapacitorDischarger.kicad_pcb (KiCad board)
At the start: 2 copper layers, 120 x 90 mm, 42 parts, among them J3 MKDS5/2-9.5, J4 MKDS5/2-9.5, J5 PM-128 input, Q1 MPSA42, Q2 STP10NK80Z

Commit message: Enclosure, front-panel LED via XH, DC-jack 9 V supply, build instructions
- mechanical/enclosure: parametric FreeCAD case for the single-sided board
  (base + screwed cover, PM-128 in the cover, sockets in line with J3/J4,
  9 V jack on the left wall with a floating-supply warning, LED on the front,
  baffled vents, snap hooks + supports for the 2-hole PCB), fit-check script
- LED1 off-board on a JST XH cable (J6); D_clamp2 (BZX55C8V2) holds LED_A at
  8.2 V if the LED is unplugged; sims 15/15 PASS; both boards re-placed, DRC clean
- PM-128 powered from any floating 9 V via a panel DC jack (battery box dropped)
- instruction.md: PCB making, assembly, wiring, tests, calibration, use

Co-Authored-By: Claude Opus 5.5 (1M context) <noreply@anthropic.com>
Parts:
- removed LED1: HLMP-4700 red, LED_THT:LED_D5.0mm
- added D_clamp2: BZX55C8V2, Diode_THT:D_DO-35_SOD27_P5.08mm_Vertical_AnodeUp, F.Cu at (139.0, 125.0)
- added J6: XH LED cable, Connector_JST:JST_XH_B2B-XH-A_1x02_P2.50mm_Vertical, F.Cu at (144.5, 128.0)
Connections:
- D_LED1 pad 2: Net-(D_LED1-A) -> /LED_A
Routing:
- net /BRIDGE_P: track 51.3 -> 39.4 mm
- net /LED_A: track 0.00 -> 10.6 mm
- net /HVp: track 133.5 -> 124.5 mm
- net Net-(D_LED1-A): track 4.88 -> 0.00 mm
- net /GND: track 299.8 -> 304.5 mm, vias 1 -> 2
- net /PROBE_A: track 27.6 -> 26.7 mm
